File: KiCad/DesignSchematic/DesignSchematic.kicad_sch (KiCad schematic)
At the start: 18 parts, among them M1 Motor_DC, M2 Motor_DC, SW1 SW_DPST, U1 EDU-CIAA, U2 AS5600, U3 AS5600, U4 MT3608, U5 VL53L0X, U6 DVR-8833, U7 MPU6050

Commit message: Esquematico
Parts:
- removed BT1, BT2: Battery_18650, symbol Device:Battery_Cell
- removed BT3: Battery 18650, symbol Device:Battery_Cell
- added C3, C4, C5, C6: 100nF, symbol Device:C
- added J1: Conn_01x02, symbol Connector_Generic:Conn_01x02
- added J2: Conn_01x02, Connector_PinSocket_2.54mm:PinSocket_1x02_P2.54mm_Vertical, symbol Connector_Generic:Conn_01x02
Connections:
- net +3.3V: now also U1.P2-01 (3V3), C3.1, C4.1, C5.1, C6.1; no longer U1.P1-01 (3V3)
- net +7.4V: no longer D2.2 (A)
- net AIN1: now also U1.P2-40 (GPIO8); no longer U1.P1-34 (T_COL2)
- net AIN2: now also U1.P2-30 (LCD1); no longer U1.P1-39 (T_COL0)
- net BIN1: now also U1.P2-28 (LCD2); no longer U1.P1-37 (T_FIL2)
- net BIN2: now also U1.P2-26 (LCD3); no longer U1.P1-35 (T_FIL3)
- net GND: now also C3.2, C4.2, C5.2, C6.2, J1.2 (Pin_2), J2.2 (Pin_2)
- net at D1.2 (A): now also J2.1 (Pin_1)
- new net: D2.2 (A), J1.1 (Pin_1)
Other:
- moved on the sheet: D1, U2, U3, U5, U7
